File: Final Project.kicad_sch (KiCad schematic)
At the start: 15 parts, among them J1 Mini-DIN-6, SW1 Button, U1 TSOP382xx, U2 ATMEGA328p-u, Y1 Crystal

Commit message: Fixed Schematic
Parts:
- removed J1: Mini-DIN-6, symbol Connector:Mini-DIN-6
- removed R1, R2: 4.7k, symbol Device:R_Small_US
Connections:
- net CLK: no longer names the net of U2.14 (PB0)
- net DATA: no longer names the net of U2.15 (PB1)
- no-connect marks 6 -> 4
Other:
- note removed: "PS/2 Interface"
